File: hardware/AD8426_PSG.kicad_sch (KiCad schematic)
At the start: 19 parts, among them U4 AD8426BCPZ-WP

Commit message: updated some docs
Parts:
- removed R20, R21, R22, R23, R24, R25: 350, symbol Device:R_45deg
- removed Rstrain1, Rstrain2: 350, symbol Device:R_Variable
- removed RwireA1, RwireA2, RwireB1, RwireB2: -, symbol Device:R_US
- renumbered C18 to C14, C19 to C15, C20 to C16, C21 to C17, U4 to U3
Connections:
- net IN1- is gone; now on net Strain1-: U3.1 (-IN1)
- net IN2- is gone; now on net Strain2-: U3.12 (-IN2)
- net Strain1-: no longer U3.4 (+IN1)
- net Strain2-: no longer U3.9 (+IN2)
- net +2V5 renamed VREF
- net +5VA renamed VAA
- new net Strain1+: U3.4 (+IN1)
- new net Strain2+: U3.9 (+IN2)
Other:
- moved on the sheet: C14, C15, C16, C17, Rg1, Rg2, U3

Commit message: finalize board before switch to stm
Parts:
- Rg1, Rg2: value 99 -> -
Other:
- note added: "AD8426 transfer func.: VOUT = G * (VIN+ - VIN-) + VREF where: G = 1 + (49.4 kΩ / RG) which rearranges to: RG = 49.4 kΩ / (G - 1) Datasheet Table 11. Gains Achieved Using 1% Resistors | 1% Standard Table Value of RG | Calculated Gain | --------------------------------------- | 49.9 kΩ | 1.990 | | 12.4 kΩ | 4.984 | | 5.49 kΩ | 9.998 | | 2.61 kΩ | 19.93 | | 1.00 kΩ | 50.40 | | 499 Ω | 100.0 | | 249 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"
Changed lines of the file:
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@@
 	(paper "A4")
 	(rectangle
-		(start 83.82 67.31)
-		(end 226.06 118.11)
+		(start 83.82 59.69)
+		(end 226.06 138.43)
 		(stroke
 			(width 0)
@@
 		(fill
 			(type none)
+		)
+	)
+	(text "AD8426 transfer func.: 	VOUT = G * (VIN+ - VIN-) + VREF\nwhere: 					G = 1 + (49.4 kΩ / RG)\nwhich rearranges to: 	RG = 49.4 kΩ / (G - 1)\n\nDatasheet Table 11. Gains Achieved Using 1% Resistors\n\n|  1% Standard Table Value of RG  |    Calculated Gain     |\n---------------------------------------\n| 49.9 kΩ					| 1.990				|\n| 12.4 kΩ					| 4.984				|\n| 5.49 kΩ					| 9.998				|\n| 2.61 kΩ					| 19.93				|\n| 1.00 kΩ					| 50.40				|\n| 499 Ω						| 100.0				|\n| 249 Ω						| 199.4				|\n| 100 Ω						| 495.0				|\n| 49.9 Ω					| 991.0				|\n* AD8426 defaults to G = 1 without a gain resistor. \nTo determine total gain accuracy, include RG's tolerance \nand drift. Without RG, gain error and drift are minimal.\n"
+		(exclude_from_sim no)
+		(at 125.222 121.666 0)
+		(effects
+			(font
+				(size 0.889 0.889)
+			)
+			(justify left)
 		)
 	)
@@
 	(wire
 		(pts
-			(xy 115.57 63.5) (xy 115.57 82.55)
+			(xy 115.57 57.15) (xy 115.57 82.55)
 		)
 		(stroke
@@
 	(wire
 		(pts
-			(xy 189.23 121.92) (xy 189.23 92.71)
+			(xy 189.23 142.24) (xy 189.23 92.71)
 		)
 		(stroke
@@
 	(wire
 		(pts
-			(xy 113.03 121.92) (xy 113.03 96.52)
+			(xy 113.03 142.24) (xy 113.03 96.52)
 		)
 		(stroke
@@
 	(wire
 		(pts
-			(xy 217.17 121.92) (xy 217.17 95.25)
+			(xy 217.17 142.24) (xy 217.17 95.25)
 		)
 		(stroke
@@
 	(wire
 		(pts
-			(xy 175.26 121.92) (xy 175.26 100.33)
+			(xy 175.26 142.24) (xy 175.26 100.33)
 		)
 		(stroke
@@
 	(wire
 		(pts
-			(xy 97.79 63.5) (xy 97.79 90.17)
+			(xy 97.79 57.15) (xy 97.79 90.17)
 		)
 		(stroke
@@
 	(wire
 		(pts
-			(xy 92.71 91.44) (xy 92.71 63.5)
-		)
-		(stroke
-			(width 0.2032)
-			(type default)
-			(color 194 0 0 1)
-		)
-	)
-	(wire
-		(pts
-			(xy 92.71 102.87) (xy 92.71 121.92)
+			(xy 92.71 91.44) (xy 92.71 57.15)
+		)
+		(stroke
+			(width 0.2032)
+			(type default)
+			(color 194 0 0 1)
+		)
+	)
+	(wire
+		(pts
+			(xy 92.71 102.87) (xy 92.71 142.24)
 		)
 		(stroke
@@
 	(wire
 		(pts
-			(xy 208.28 82.55) (xy 208.28 63.5)
+			(xy 208.28 82.55) (xy 208.28 57.15)
 		)
 		(stroke
@@
 	(hierarchical_label "Strain2-"
 		(shape input)
-		(at 189.23 121.92 270)
+		(at 189.23 142.24 270)
 		(effects
 			(font
@@
 	(hierarchical_label "Strain1-"
 		(shape input)
-		(at 115.57 63.5 90)
+		(at 115.57 57.15 90)
 		(effects
 			(font
@@
 	(hierarchical_label "VAA"
 		(shape input)
-		(at 92.71 63.5 90)
+		(at 92.71 57.15 90)
 		(effects
 			(font
@@
 	(hierarchical_label "GNDA"
 		(shape input)
-		(at 92.71 121.92 270)
+		(at 92.71 142.24 270)
 		(effects
 			(font
@@
 	(hierarchical_label "GNDA"
 		(shape input)
-		(at 217.17 121.92 270)
+		(at 217.17 142.24 270)
 		(effects
 			(font
@@
 	(hierarchical_label "Strain1+"
 		(shape input)
-		(at 97.79 63.5 90)
+		(at 97.79 57.15 90)
 		(effects
 			(font
@@
 	(hierarchical_label "VAA"
 		(shape input)
-		(at 208.28 63.5 90)
+		(at 208.28 57.15 90)
 		(effects
 			(font
@@
 	(hierarchical_label "Strain2+"
 		(shape input)
-		(at 175.26 121.92 270)
+		(at 175.26 142.24 270)
 		(effects
 			(font
@@
 	(hierarchical_label "VREF"
 		(shape input)
-		(at 113.03 121.92 270)
+		(at 113.03 142.24 270)
 		(effects
 			(font
@@
 			)
 		)
-		(property "Value" "99"
+		(property "Value" "-"
 			(at 107.95 82.804 90)
 			(effects
@@
 		(on_board yes)
 		(dnp no)
-		(fields_autoplaced yes)
 		(property "Reference" "U3"
 			(at 147.32 72.39 0)
@@
 			)
 		)
-		(property "Value" "99"
+		(property "Value" "-"
 			(at 181.61 100.076 90)
 			(effects
