File: hardware/AD8426_PSG.kicad_sch (KiCad schematic)
At the start: 7 parts, among them U4 AD8426BCPZ-WP

Commit message: chore(hw): migrate KiCad files to the KiCad 10 format
Via `kicad-cli sch upgrade` / `pcb upgrade` (bread-infra
scripts/upgrade_kicad10.sh). Verified lossless: identical netlist, footprint
positions and routing.

Note `sch upgrade` does not cascade into hierarchical sub-sheets, so every
.kicad_sch is upgraded individually -- upgrading only the root sheet leaves
sub-sheets on the old format, which looks migrated and is not.
Parts:
- renumbered C16 to C24, C17 to C25, C18 to C26, C19 to C27, Rg1 to Rg5, Rg2 to Rg6, U4 to U6

Commit message: fix(hw): re-point stale library nicknames
These parts exist in KiCad-Master-Lib; the boards referenced libraries that no
longer exist (kml-custom, KML-Custom, and SparkFun libraries that never
contained the part) or names the library has since changed.

KiCad embeds footprint geometry in the .kicad_pcb, so the boards rendered and
fabricated correctly and the rot stayed invisible -- it only surfaces on
update-from-library, or when a generator tries to resolve a nickname.

Nickname/name only. No geometry is changed:

  SparkFun-DiscreteSemi:AP63205 -> KMLib_IC_Power:AP63205WU-7_Buck_Regulator
  SparkFun-LED:WS2812-5050-4PIN -> KMLib_IC_SMD:WS2812-5050-4PIN
  kml-custom:1439890 -> KMLib_Connectors:1439890
  kml-custom:AD8426BCPZ-WP -> KMLib_IC_Analog:AD8426BCPZ-WP_Instrumentation_Amplifier
  kml-custom:ADS131M08IPBS -> KMLib_IC_Analog:ADS131M08IPBS_24-bit_ADC
  kml-custom:CP_16_19_ADI -> KMLib_IC_SMD:CP_16_19_ADI
  kml-custom:DGN8_1P89X1P57 -> KMLib_IC_SMD:DGN8_1P89X1P57
  kml-custom:Full_Bridge_Strain_Gauge -> KMLib_Sensors:Full_Bridge_Strain_Gauge
  kml-custom:MODULE_NUCLEO-L432KC -> KMLib_Boards_Modules:MODULE_NUCLEO-L432KC
  kml-custom:NUCLEO-L432KC -> KMLib_IC_MCU_MPU:NUCLEO-L432KC
  kml-custom:QFP50P700X700X120-32N -> KMLib_IC_SMD:QFP50P700X700X120-32N
  kml-custom:TPS7A4901DGNR -> KMLib_IC_Power:TPS7A4901DGNR_LDO_Regulator
  kml-custom:Thermal Pad -> KMLib_Mounting:Thermal_Pad

Only references that failed to resolve were touched. Generic parts (<=4 pins)
and KiCad *-rescue libraries are deliberately excluded: fingerprint matching
cannot distinguish a 2-pin resistor from a 2-pin capacitor, so those are being
done by hand.
Parts:
- U6: footprint kml-custom:CP_16_19_ADI -> KMLib_IC_SMD:CP_16_19_ADI; symbol kml-custom:AD8426BCPZ-WP -> KMLib_IC_Analog:AD8426BCPZ-WP_Instrumentation_Amplifier
Changed lines of the file:
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@@
 	)
 	(symbol
-		(lib_id "kml-custom:AD8426BCPZ-WP")
+		(lib_id "KMLib_IC_Analog:AD8426BCPZ-WP_Instrumentation_Amplifier")
 		(at 127 82.55 0)
 		(unit 1)
@@
 			)
 		)
-		(property "Footprint" "kml-custom:CP_16_19_ADI"
+		(property "Footprint" "KMLib_IC_SMD:CP_16_19_ADI"
 			(at 127 82.55 0)
 			(hide yes)
