File: hardware/BREAD_Slice.kicad_pcb (KiCad board)
At the start: 4 copper layers, 100.1 x 100 mm, 107 parts, among them IC1 ADS131M08IPBS, J1 Conn_01x10_Female, J10 Micro_SD_Card, J2 1439890, J3 1439890, J4 1439890, J5 1439890, J6 1439890, J7 1439890, J8 1439890, J9 1439890, U1 AP63205, U2 NUCLEO-L432KC, U3 MCP6022, U4 AD8426BCPZ-WP, U5 AD8426BCPZ-WP, U6 AD8426BCPZ-WP, U7 AD8426BCPZ-WP, U8 TPS7A4901DGNR, U9 TPS7A4901DGNR

Commit message: fix(hw): re-point stale library nicknames
These parts exist in KiCad-Master-Lib; the boards referenced libraries that no
longer exist (kml-custom, KML-Custom, and SparkFun libraries that never
contained the part) or names the library has since changed.

KiCad embeds footprint geometry in the .kicad_pcb, so the boards rendered and
fabricated correctly and the rot stayed invisible -- it only surfaces on
update-from-library, or when a generator tries to resolve a nickname.

Nickname/name only. No geometry is changed:

  SparkFun-DiscreteSemi:AP63205 -> KMLib_IC_Power:AP63205WU-7_Buck_Regulator
  SparkFun-LED:WS2812-5050-4PIN -> KMLib_IC_SMD:WS2812-5050-4PIN
  kml-custom:1439890 -> KMLib_Connectors:1439890
  kml-custom:AD8426BCPZ-WP -> KMLib_IC_Analog:AD8426BCPZ-WP_Instrumentation_Amplifier
  kml-custom:ADS131M08IPBS -> KMLib_IC_Analog:ADS131M08IPBS_24-bit_ADC
  kml-custom:CP_16_19_ADI -> KMLib_IC_SMD:CP_16_19_ADI
  kml-custom:DGN8_1P89X1P57 -> KMLib_IC_SMD:DGN8_1P89X1P57
  kml-custom:Full_Bridge_Strain_Gauge -> KMLib_Sensors:Full_Bridge_Strain_Gauge
  kml-custom:MODULE_NUCLEO-L432KC -> KMLib_Boards_Modules:MODULE_NUCLEO-L432KC
  kml-custom:NUCLEO-L432KC -> KMLib_IC_MCU_MPU:NUCLEO-L432KC
  kml-custom:QFP50P700X700X120-32N -> KMLib_IC_SMD:QFP50P700X700X120-32N
  kml-custom:TPS7A4901DGNR -> KMLib_IC_Power:TPS7A4901DGNR_LDO_Regulator
  kml-custom:Thermal Pad -> KMLib_Mounting:Thermal_Pad

Only references that failed to resolve were touched. Generic parts (<=4 pins)
and KiCad *-rescue libraries are deliberately excluded: fingerprint matching
cannot distinguish a 2-pin resistor from a 2-pin capacitor, so those are being
done by hand.
Parts:
- D1: footprint SparkFun-LED:WS2812-5050-4PIN -> KMLib_IC_SMD:WS2812-5050-4PIN
- HS1: footprint kml-custom:Thermal Pad -> KMLib_Mounting:Thermal_Pad
- IC1: footprint kml-custom:QFP50P700X700X120-32N -> KMLib_IC_SMD:QFP50P700X700X120-32N
- J2, J3, J4, J5, J6, J7, J8, J9: footprint kml-custom:1439890 -> KMLib_Connectors:1439890
- U2: footprint kml-custom:MODULE_NUCLEO-L432KC -> KMLib_Boards_Modules:MODULE_NUCLEO-L432KC
- U4, U5, U6, U7: footprint kml-custom:CP_16_19_ADI -> KMLib_IC_SMD:CP_16_19_ADI
- U8, U9: footprint kml-custom:DGN8_1P89X1P57 -> KMLib_IC_SMD:DGN8_1P89X1P57
Changed lines of the file:
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@@
 		(embedded_fonts no)
 	)
-	(footprint "kml-custom:MODULE_NUCLEO-L432KC"
+	(footprint "KMLib_Boards_Modules:MODULE_NUCLEO-L432KC"
 		(layer "F.Cu")
 		(at 85.09 155.305)
@@
 		)
 	)
-	(footprint "kml-custom:DGN8_1P89X1P57"
+	(footprint "KMLib_IC_SMD:DGN8_1P89X1P57"
 		(layer "F.Cu")
 		(at 74.6 120.75 180)
@@
 		)
 	)
-	(footprint "kml-custom:Thermal Pad"
+	(footprint "KMLib_Mounting:Thermal_Pad"
 		(layer "F.Cu")
 		(at 66.774465 162.653932)
@@
 		)
 	)
-	(footprint "kml-custom:1439890"
+	(footprint "KMLib_Connectors:1439890"
 		(layer "F.Cu")
 		(at 126.48 168.715)
@@
 		)
 	)
-	(footprint "kml-custom:CP_16_19_ADI"
+	(footprint "KMLib_IC_SMD:CP_16_19_ADI"
 		(layer "F.Cu")
 		(at 131.25 103.15 90)
@@
 		)
 	)
-	(footprint "kml-custom:1439890"
+	(footprint "KMLib_Connectors:1439890"
 		(layer "F.Cu")
 		(at 143.505 106.755 90)
@@
 		)
 	)
-	(footprint "SparkFun-LED:WS2812-5050-4PIN"
+	(footprint "KMLib_IC_SMD:WS2812-5050-4PIN"
 		(locked yes)
 		(layer "F.Cu")
@@
 		)
 	)
-	(footprint "kml-custom:1439890"
+	(footprint "KMLib_Connectors:1439890"
 		(layer "F.Cu")
 		(at 143.53 128.83 90)
@@
 		)
 	)
-	(footprint "kml-custom:CP_16_19_ADI"
+	(footprint "KMLib_IC_SMD:CP_16_19_ADI"
 		(layer "F.Cu")
 		(at 135.1875 157.2625)
@@
 		)
 	)
-	(footprint "kml-custom:1439890"
+	(footprint "KMLib_Connectors:1439890"
 		(layer "F.Cu")
 		(at 148.545 168.73)
@@
 		)
 	)
-	(footprint "kml-custom:QFP50P700X700X120-32N"
+	(footprint "KMLib_IC_SMD:QFP50P700X700X120-32N"
 		(layer "F.Cu")
 		(at 111.125 125.9 180)
@@
 		)
 	)
-	(footprint "kml-custom:1439890"
+	(footprint "KMLib_Connectors:1439890"
 		(layer "F.Cu")
 		(at 144.03 93.345 180)
@@
 		)
 	)
-	(footprint "kml-custom:1439890"
+	(footprint "KMLib_Connectors:1439890"
 		(layer "F.Cu")
 		(at 143.53 150.905 90)
@@
 		)
 	)
-	(footprint "kml-custom:CP_16_19_ADI"
+	(footprint "KMLib_IC_SMD:CP_16_19_ADI"
 		(layer "F.Cu")
 		(at 131.575 142.008948 90)
@@
 		)
 	)
-	(footprint "kml-custom:1439890"
+	(footprint "KMLib_Connectors:1439890"
 		(layer "F.Cu")
 		(at 121.955 93.345 180)
@@
 		)
 	)
-	(footprint "kml-custom:DGN8_1P89X1P57"
+	(footprint "KMLib_IC_SMD:DGN8_1P89X1P57"
 		(layer "F.Cu")
 		(at 74.3795 106.400001 180)
@@
 		)
 	)
-	(footprint "kml-custom:1439890"
+	(footprint "KMLib_Connectors:1439890"
 		(layer "F.Cu")
 		(at 99.88 93.345 180)
@@
 		)
 	)
-	(footprint "kml-custom:CP_16_19_ADI"
+	(footprint "KMLib_IC_SMD:CP_16_19_ADI"
 		(layer "F.Cu")
 		(at 113.074999 104.9653 180)
