File: hardware/BREAD_Slice.kicad_sch (KiCad schematic)
At the start: 14 parts, among them J1 Conn_01x10_Female

Commit message: initial commit of hw
Parts:
- added C10, C11, C12, C14, C15, C5, C6, C7, C8, C9: 10n, Capacitor_SMD:C_1206_3216Metric, symbol Device:C_Small
- added C13, C16: 10u, Capacitor_SMD:C_1206_3216Metric, symbol Device:C_Small
- added C17: 220n, Capacitor_SMD:C_1206_3216Metric, symbol Device:C_Small
- added IC1: ADS131M08IPBS, QFP50P700X700X120-32N, symbol kml-custom:ADS131M08IPBS
- added J2, J3, J4, J5: Screw_Terminal_01x04, symbol Connector:Screw_Terminal_01x04
- added R1, R10, R11, R12, R13, R14, R15, R16, R2, R3, R4, R5, R6, R7, R8, R9: 1k, symbol Device:R
- added R17, R18: 99, symbol Device:R
- added R19: 2500, symbol Device:R
- added U2: TPS7A4901DGNR, DGN8_1P89X1P57, symbol kml-custom:TPS7A4901DGNR
- added U3: LM4040AIM3-2.5/NOPB, DBZ3, symbol kml-custom:LM4040AIM3-2.5_NOPB
- added Y1: ACO-xxxMHz, Oscillator:Oscillator_DIP-14, symbol Oscillator:ACO-xxxMHz
Connections:
- net +12V: now also C13.2, U2.5 (EN), U2.8 (IN)
- net +5V: now also IC1.26 (DVDD), Y1.14 (Vcc)
- net E_STOP: no longer A1.5 (D2)
- net GND: now also C13.1, C14.1, C16.1, C17.1, IC1.13 (AGND_1), IC1.14 (REFIN), IC1.25 (DGND), IC1.28 (AGND_2), R10.2, R12.2, R14.2, R16.2, R18.1, R2.2, R4.2, R6.2, R8.2, U2.3 (NC), U2.4 (GND), U2.EPAD, U3.2 (ANODE), Y1.7 (GND)
- net RESET: now also IC1.16 (~{SYNC}/~{RESET})
- net D10 renamed SS
- net SS: now also IC1.17 (~{CS})
- net D11 renamed MOSI
- net MOSI: now also IC1.21 (DIN)
- net D12 renamed MISO
- net MISO: now also IC1.20 (DOUT)
- net D13 renamed SCK
- net SCK: now also IC1.19 (SCLK)
- net D9 renamed DRDY
- net DRDY: now also IC1.18 (~{DRDY})
- net INT: no longer names the net of J1.7 (Pin_7)
- net INT: no longer A1.6 (D3)
- new net: C15.1, R17.1, R18.2, U2.2 (FB)
- new net: C14.2, U2.6 (NR/SS)
- new net: C17.2, IC1.24 (CAP)
- new net +2V5: R19.2, U3.1 (CATHODE)
- new net +5VA: C15.2, C16.2, IC1.15 (AVDD), R17.2, R19.1, U2.1 (OUT)
- new net AD8426 Dual Precision Strain Gauge1/Strain1+: J2.4 (Pin_4)
- new net AD8426 Dual Precision Strain Gauge1/Strain1-: J2.3 (Pin_3)
- new net AD8426 Dual Precision Strain Gauge1/Strain2+: J2.2 (Pin_2)
- new net AD8426 Dual Precision Strain Gauge1/Strain2-: J2.1 (Pin_1)
- new net AD8426 Dual Precision Strain Gauge2/Strain1+: J3.4 (Pin_4)
- new net AD8426 Dual Precision Strain Gauge2/Strain1-: J3.3 (Pin_3)
- new net AD8426 Dual Precision Strain Gauge2/Strain2+: J3.2 (Pin_2)
- new net AD8426 Dual Precision Strain Gauge2/Strain2-: J3.1 (Pin_1)
- new net AD8426 Dual Precision Strain Gauge3/Strain1+: J4.4 (Pin_4)
- new net AD8426 Dual Precision Strain Gauge3/Strain1-: J4.3 (Pin_3)
- new net AD8426 Dual Precision Strain Gauge3/Strain2+: J4.2 (Pin_2)
- new net AD8426 Dual Precision Strain Gauge3/Strain2-: J4.1 (Pin_1)
- new net AD8426 Dual Precision Strain Gauge4/Strain1+: J5.4 (Pin_4)
- new net AD8426 Dual Precision Strain Gauge4/Strain1-: J5.3 (Pin_3)
- new net AD8426 Dual Precision Strain Gauge4/Strain2+: J5.2 (Pin_2)
- new net AD8426 Dual Precision Strain Gauge4/Strain2-: J5.1 (Pin_1)
- new net CLK_8MHz: A1.5 (D2), IC1.23 (XTAL1/CLKIN), Y1.8 (OUT)
- new net ESTOP: A1.6 (D3)
- new net IN0+: C5.2, IC1.30 (AIN0N), R1.1
- new net IN0-: C5.1, IC1.29 (AIN0P), R2.1
- new net IN1+: C6.2, IC1.32 (AIN1P), R3.1
- new net IN1-: C6.1, IC1.31 (AIN1N), R4.1
- new net IN2+: C7.2, IC1.1 (AIN2P), R5.1
- new net IN2-: C7.1, IC1.2 (AIN2N), R6.1
- new net IN3+: C8.2, IC1.3 (AIN3N), R7.1
- new net IN3-: C8.1, IC1.4 (AIN3P), R8.1
- new net IN4+: C9.2, IC1.5 (AIN4P), R9.1
- new net IN4-: C9.1, IC1.6 (AIN4N), R10.1
- new net IN5+: C10.2, IC1.7 (AIN5N), R11.1
- new net IN5-: C10.1, IC1.8 (AIN5P), R12.1
- new net IN6+: C11.2, IC1.9 (AIN6P), R13.1
- new net IN6-: C11.1, IC1.10 (AIN6N), R14.1
- new net IN7+: C12.2, IC1.11 (AIN7N), R15.1
- new net IN7-: C12.1, IC1.12 (AIN7P), R16.1
- new net OUT0: R1.2
- new net OUT1: R13.2, R3.2
- new net OUT2: R11.2, R15.2, R5.2
- new net OUT3: R7.2
- new net OUT4: R9.2
- no-connect marks 6 -> 11
Other:
- added sheet AD8426 Dual Precision Strain Gauge1 (AD8426_PSG.kicad_sch)
- added sheet AD8426 Dual Precision Strain Gauge2 (AD8426_PSG.kicad_sch)
- added sheet AD8426 Dual Precision Strain Gauge3 (AD8426_PSG.kicad_sch)
- added sheet AD8426 Dual Precision Strain Gauge4 (AD8426_PSG.kicad_sch)
- note added: "8MHz External Clock"
- note added: "ADC 24-bit 32-kSPS"
- note added: "Analog 2v5"
- note added: "Analog 5V"
- note added: "Antialiasing"
- note added: "Connect EPAD to GND plane using multiple vias"
- note added: "D2 corresponds to PA00 which is EXTCLK on ATMega809 will need fuse changed and appropriate programmer"
- note added: "Digital 5V"
- note added: "For DVDD > 2.7 V, connect 220 nF from CAP to DGND. For DVDD ≤ 2 V, tie CAP to DVDD and use 100 nF to DGND for decoupling."
- note added: "removed int to move estop to make room on D2"
- note added: "x8 Wheatstone Bridge + Instrumentation Amp"

Commit message: updated some docs
Parts:
- removed C13, C16: 10u, Capacitor_SMD:C_1206_3216Metric, symbol Device:C_Small
- removed C14, C15: 10n, Capacitor_SMD:C_1206_3216Metric, symbol Device:C_Small
- removed D1: WS2812B_5050, SparkFun-LED:WS2812-5050-4PIN, symbol SparkFun-LED:WS2812B_5050
- removed HS1: Heatsink_Pad, KML-Custom:Thermal Pad, symbol Mechanical:Heatsink_Pad
- removed R19: 2500, symbol Device:R
- removed U2: TPS7A4901DGNR, DGN8_1P89X1P57, symbol kml-custom:TPS7A4901DGNR
- removed U3: LM4040AIM3-2.5/NOPB, DBZ3, symbol kml-custom:LM4040AIM3-2.5_NOPB
- added D2: WS2812B_5050, SparkFun-LED:WS2812-5050-4pin, symbol SparkFun-LED:WS2812B_5050
- added HS2: Heatsink_Pad_2Pin, symbol Mechanical:Heatsink_Pad_2Pin
- added J6, J7, J8, J9: Screw_Term_01x04, symbol Connector:Screw_Terminal_01x04
- added RSG1, RSG2, RSG4, RSG5: 350, symbol kml-custom:Full Bridge Strain Gauge
- added RSG3: 480, symbol kml-custom:Full Bridge Strain Gauge
- added RSG6: 700, symbol kml-custom:Full Bridge Strain Gauge
- added RSG7, RSG8: 300, symbol kml-custom:Full Bridge Strain Gauge
- added U2: OP1177ARM, Package_SO:MSOP-8_3x3mm_P0.65mm, symbol Amplifier_Operational:OP1177ARM
- J2, J3, J4, J5: value Screw_Terminal_01x04 -> Screw_Term_01x04
- R17, R18: value 99 -> 50k
- U1: value ~ -> AP63205
- renumbered C17 to C13
Connections:
- net AD8426 Dual Precision Strain Gauge2/Strain1+ is gone; now on net +5VA: J3.4 (Pin_4)
- net AD8426 Dual Precision Strain Gauge2/Strain1- is gone; now on net AD8426 x2 Strain Gauge1/Strain2+: J3.3 (Pin_3)
- net AD8426 Dual Precision Strain Gauge2/Strain2+ is gone; now on net GNDA: J3.2 (Pin_2)
- net AD8426 Dual Precision Strain Gauge2/Strain2- is gone; now on net AD8426 x2 Strain Gauge1/Strain2-: J3.1 (Pin_1)
- net AD8426 Dual Precision Strain Gauge3/Strain2+ is gone; now on net GNDA: J4.2 (Pin_2)
- net AD8426 Dual Precision Strain Gauge4/Strain1+ is gone; now on net +5VA: J5.4 (Pin_4)
- net AD8426 Dual Precision Strain Gauge4/Strain2+ is gone; now on net GNDA: J5.2 (Pin_2)
- net +5V: now also D2.1 (VDD); no longer C3.2, C4.2, L1.2, U1.1 (FB), Y1.14 (Vcc)
- net +5VA: now also Y1.14 (Vcc), J7.4 (Pin_4), J9.4 (Pin_4), RSG2. (SIG+), RSG4. (SIG+), RSG6. (SIG+), RSG8. (SIG+); no longer IC1.15 (AVDD), R17.2
- net AD8426 x2 Strain Gauge1/Strain1+: now also J2.3 (Pin_3), RSG1. (SIG+); no longer J2.4 (Pin_4)
- net AD8426 x2 Strain Gauge1/Strain1-: now also J2.1 (Pin_1), RSG1. (SIG+); no longer J2.3 (Pin_3)
- net AD8426 x2 Strain Gauge1/Strain2+: now also RSG2. (SIG+); no longer J2.2 (Pin_2)
- net AD8426 x2 Strain Gauge1/Strain2-: now also RSG2. (SIG+); no longer J2.1 (Pin_1)
- net GND: now also D2.3 (VSS), HS2.1; no longer A1.29 (GND), A1.4 (GND), C1.1, C13.1, C3.1, C4.1, IC1.13 (AGND_1), IC1.14 (REFIN), IC1.25 (DGND), IC1.28 (AGND_2), R10.2, R12.2, R14.2, R16.2, R18.1, R2.2, R4.2, R6.2, R8.2, U1.4 (GND), Y1.7 (GND)
- net LED: now also D2.4 (DIN)
- net OUT0: now also R11.2, R13.2, R15.2, R3.2, R5.2, R7.2, R9.2
- net OUT1: no longer R13.2, R3.2
- net OUT2: no longer R11.2, R15.2, R5.2
- net OUT3: no longer R7.2
- net OUT4: no longer R9.2
- net GNDA: now reaches R18.2
- net GNDA: now also IC1.13 (AGND_1), IC1.14 (REFIN), IC1.28 (AGND_2), J2.2 (Pin_2), R10.2, R12.2, R14.2, R16.2, R2.2, R4.2, R6.2, R8.2, Y1.7 (GND), J6.2 (Pin_2), J7.2 (Pin_2), J8.2 (Pin_2), J9.2 (Pin_2), RSG1. (SIG+), RSG2. (SIG+), RSG3. (SIG+), RSG4. (SIG+), RSG5. (SIG+), RSG6. (SIG+), RSG7. (SIG+), RSG8. (SIG+), U2.4 (V-); no longer R17.1
- net AD8426 Dual Precision Strain Gauge3/Strain1+ renamed VAA
- net VAA: now also IC1.15 (AVDD), J2.4 (Pin_4), R17.1, J6.4 (Pin_4), J8.4 (Pin_4), RSG1. (SIG+), RSG3. (SIG+), RSG5. (SIG+), RSG7. (SIG+), U2.7 (V+)
- net AD8426 Dual Precision Strain Gauge3/Strain1- renamed AD8426 x2 Strain Gauge2/Strain1+
- net AD8426 x2 Strain Gauge2/Strain1+: now also RSG3. (SIG+)
- net AD8426 Dual Precision Strain Gauge3/Strain2- renamed AD8426 x2 Strain Gauge2/Strain1-
- net AD8426 x2 Strain Gauge2/Strain1-: now also RSG3. (SIG+)
- net AD8426 Dual Precision Strain Gauge4/Strain1- renamed AD8426 x2 Strain Gauge2/Strain2+
- net AD8426 x2 Strain Gauge2/Strain2+: now also RSG4. (SIG+)
- net AD8426 Dual Precision Strain Gauge4/Strain2- renamed AD8426 x2 Strain Gauge2/Strain2-
- net AD8426 x2 Strain Gauge2/Strain2-: now also RSG4. (SIG+)
- new net: R17.2, R18.1, U2.3 (+)
- new net +5VD: C3.2, C4.2, L1.2, U1.1 (FB)
- new net AD8426 x2 Strain Gauge3/Strain1+: J6.3 (Pin_3), RSG5. (SIG+)
- new net AD8426 x2 Strain Gauge3/Strain1-: J6.1 (Pin_1), RSG5. (SIG+)
- new net AD8426 x2 Strain Gauge3/Strain2+: J7.3 (Pin_3), RSG6. (SIG+)
- new net AD8426 x2 Strain Gauge3/Strain2-: J7.1 (Pin_1), RSG6. (SIG+)
- new net AD8426 x2 Strain Gauge4/Strain1+: J8.3 (Pin_3), RSG7. (SIG+)
- new net AD8426 x2 Strain Gauge4/Strain1-: J8.1 (Pin_1), RSG7. (SIG+)
- new net AD8426 x2 Strain Gauge4/Strain2+: J9.3 (Pin_3), RSG8. (SIG+)
- new net AD8426 x2 Strain Gauge4/Strain2-: J9.1 (Pin_1), RSG8. (SIG+)
- new net GNDD: A1.29 (GND), A1.4 (GND), C1.1, C13.1, C3.1, C4.1, HS2.2, IC1.25 (DGND), U1.4 (GND)
- new net VMID: U2.2 (-), U2.6
- no-connect marks 11 -> 9
Other:
- sheet AD8426 Dual Precision Strain Gauge1 renamed AD8426 x2 Strain Gauge1
- removed sheet AD8426 Dual Precision Strain Gauge2
- removed sheet AD8426 Dual Precision Strain Gauge3
- removed sheet AD8426 Dual Precision Strain Gauge4
- added sheet AD8426 x2 Strain Gauge2 (AD8426_PSG.kicad_sch)
- added sheet AD8426 x2 Strain Gauge3 (AD8426_PSG.kicad_sch)
- added sheet AD8426 x2 Strain Gauge4 (AD8426_PSG.kicad_sch)
- added sheet TPS7A4901-5VA (tps7a4901.kicad_sch)
- added sheet TPS7A4901-VAA (tps7a4901.kicad_sch)
- sheet AD8426 x2 Strain Gauge1 ports: added GNDA, VAA, VREF; removed none
- note added: "8MHz Ext Clock"
- note added: "Adjustable analog frontend reference"
- note added: "Analog Supplies"
- note added: "Analog frontend midsupply reference"
- note added: "Arduino Nano Every ATMega 4809"
- note added: "Backplane Conn."
- note added: "Clean 5V TLL supply for external clock"
- note added: "Color Scheme Legend: ---------------------------------------------------------- color - value - reference ---------------------------------------------------------- • Red - red3 - Analog 5V Supply (e.g., for amps, ADC, references) • Brown - orange1 - Analog Ground (sensor/amp/ADC ground) • Orange - orange3 - Digital 5V Supply (MCU, digital circuits) • Black - black - Digital Ground (MCU ground) •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"
- note added: "D2 corresponds to PA00 which is EXTCLK on ATMega4809 will need fuse changed and appropriate programmer"
- note added: "Instrumentation Amp x8"
- note added: "Load Cells x8"
- note added: "Mounting Holes"
- note added: "RGB LED"
- note added: "internal note: removed int to move estop to make room on D2"
- note removed: "8MHz External Clock"
- note removed: "Analog 2v5"
- note removed: "Analog 5V"
- note removed: "Connect EPAD to GND plane using multiple vias"
- note removed: "D2 corresponds to PA00 which is EXTCLK on ATMega809 will need fuse changed and appropriate programmer"
- note removed: "removed int to move estop to make room on D2"
- note removed: "x8 Wheatstone Bridge + Instrumentation Amp"
- moved on the sheet: A1, C1, C13, C2, C3, C4, C5, H1, H2, H3, H4, IC1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
