File: hardware/BREAD_Slice.kicad_sch (KiCad schematic)
At the start: 57 parts, among them IC1 ADS131M08IPBS, J1 Conn_01x10_Female, J10 Micro_SD_Card, J2 1439890, J3 1439890, J4 1439890, J5 1439890, J6 1439890, J7 1439890, J8 1439890, J9 1439890, U1 AP63205, U2 NUCLEO-L432KC, U3 MCP6022

Commit message: fix(hw): re-point stale library nicknames
These parts exist in KiCad-Master-Lib; the boards referenced libraries that no
longer exist (kml-custom, KML-Custom, and SparkFun libraries that never
contained the part) or names the library has since changed.

KiCad embeds footprint geometry in the .kicad_pcb, so the boards rendered and
fabricated correctly and the rot stayed invisible -- it only surfaces on
update-from-library, or when a generator tries to resolve a nickname.

Nickname/name only. No geometry is changed:

  SparkFun-DiscreteSemi:AP63205 -> KMLib_IC_Power:AP63205WU-7_Buck_Regulator
  SparkFun-LED:WS2812-5050-4PIN -> KMLib_IC_SMD:WS2812-5050-4PIN
  kml-custom:1439890 -> KMLib_Connectors:1439890
  kml-custom:AD8426BCPZ-WP -> KMLib_IC_Analog:AD8426BCPZ-WP_Instrumentation_Amplifier
  kml-custom:ADS131M08IPBS -> KMLib_IC_Analog:ADS131M08IPBS_24-bit_ADC
  kml-custom:CP_16_19_ADI -> KMLib_IC_SMD:CP_16_19_ADI
  kml-custom:DGN8_1P89X1P57 -> KMLib_IC_SMD:DGN8_1P89X1P57
  kml-custom:Full_Bridge_Strain_Gauge -> KMLib_Sensors:Full_Bridge_Strain_Gauge
  kml-custom:MODULE_NUCLEO-L432KC -> KMLib_Boards_Modules:MODULE_NUCLEO-L432KC
  kml-custom:NUCLEO-L432KC -> KMLib_IC_MCU_MPU:NUCLEO-L432KC
  kml-custom:QFP50P700X700X120-32N -> KMLib_IC_SMD:QFP50P700X700X120-32N
  kml-custom:TPS7A4901DGNR -> KMLib_IC_Power:TPS7A4901DGNR_LDO_Regulator
  kml-custom:Thermal Pad -> KMLib_Mounting:Thermal_Pad

Only references that failed to resolve were touched. Generic parts (<=4 pins)
and KiCad *-rescue libraries are deliberately excluded: fingerprint matching
cannot distinguish a 2-pin resistor from a 2-pin capacitor, so those are being
done by hand.
Parts:
- D1: footprint SparkFun-LED:WS2812-5050-4PIN -> KMLib_IC_SMD:WS2812-5050-4PIN
- HS1: footprint kml-custom:Thermal Pad -> KMLib_Mounting:Thermal_Pad
- IC1: footprint kml-custom:QFP50P700X700X120-32N -> KMLib_IC_SMD:QFP50P700X700X120-32N; symbol kml-custom:ADS131M08IPBS -> KMLib_IC_Analog:ADS131M08IPBS_24-bit_ADC
- J2, J3, J4, J5, J6, J7, J8, J9: symbol kml-custom:1439890 -> KMLib_Connectors:1439890
- U1: symbol SparkFun-DiscreteSemi:AP63205 -> KMLib_IC_Power:AP63205WU-7_Buck_Regulator
- U2: footprint kml-custom:MODULE_NUCLEO-L432KC -> KMLib_Boards_Modules:MODULE_NUCLEO-L432KC; symbol kml-custom:NUCLEO-L432KC -> KMLib_IC_MCU_MPU:NUCLEO-L432KC
Changed lines of the file:
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@@
 			)
 		)
-		(property "Footprint" "kml-custom:Thermal Pad"
+		(property "Footprint" "KMLib_Mounting:Thermal_Pad"
 			(at 35.8648 95.25 0)
 			(hide yes)
@@
 	)
 	(symbol
-		(lib_id "kml-custom:1439890")
+		(lib_id "KMLib_Connectors:1439890")
 		(at 117.602 76.962 0)
 		(mirror y)
@@
 	)
 	(symbol
-		(lib_id "SparkFun-DiscreteSemi:AP63205")
+		(lib_id "KMLib_IC_Power:AP63205WU-7_Buck_Regulator")
 		(at 35.56 71.12 0)
 		(unit 1)
@@
 			)
 		)
-		(property "Footprint" "SparkFun-LED:WS2812-5050-4PIN"
+		(property "Footprint" "KMLib_IC_SMD:WS2812-5050-4PIN"
 			(at 13.97 40.64 0)
 			(hide yes)
@@
 	)
 	(symbol
-		(lib_id "kml-custom:1439890")
+		(lib_id "KMLib_Connectors:1439890")
 		(at 117.602 163.322 0)
 		(mirror y)
@@
 	)
 	(symbol
-		(lib_id "kml-custom:1439890")
+		(lib_id "KMLib_Connectors:1439890")
 		(at 99.822 55.372 0)
 		(unit 1)
@@
 	)
 	(symbol
-		(lib_id "kml-custom:1439890")
+		(lib_id "KMLib_Connectors:1439890")
 		(at 117.602 33.782 0)
 		(mirror y)
@@
 	)
 	(symbol
-		(lib_id "kml-custom:ADS131M08IPBS")
+		(lib_id "KMLib_IC_Analog:ADS131M08IPBS_24-bit_ADC")
 		(at 222.25 52.07 0)
 		(unit 1)
@@
 			)
 		)
-		(property "Footprint" "kml-custom:QFP50P700X700X120-32N"
+		(property "Footprint" "KMLib_IC_SMD:QFP50P700X700X120-32N"
 			(at 256.54 136.83 0)
 			(hide yes)
@@
 	)
 	(symbol
-		(lib_id "kml-custom:1439890")
+		(lib_id "KMLib_Connectors:1439890")
 		(at 99.822 141.732 0)
 		(unit 1)
@@
 	)
 	(symbol
-		(lib_id "kml-custom:NUCLEO-L432KC")
+		(lib_id "KMLib_IC_MCU_MPU:NUCLEO-L432KC")
 		(at 40.64 172.72 0)
 		(unit 2)
@@
 			)
 		)
-		(property "Footprint" "kml-custom:MODULE_NUCLEO-L432KC"
+		(property "Footprint" "KMLib_Boards_Modules:MODULE_NUCLEO-L432KC"
 			(at 40.64 172.72 0)
 			(hide yes)
@@
 	)
 	(symbol
-		(lib_id "kml-custom:NUCLEO-L432KC")
+		(lib_id "KMLib_IC_MCU_MPU:NUCLEO-L432KC")
 		(at 40.64 135.89 0)
 		(unit 1)
@@
 			)
 		)
-		(property "Footprint" "kml-custom:MODULE_NUCLEO-L432KC"
+		(property "Footprint" "KMLib_Boards_Modules:MODULE_NUCLEO-L432KC"
 			(at 40.64 135.89 0)
 			(hide yes)
@@
 	)
 	(symbol
-		(lib_id "kml-custom:1439890")
+		(lib_id "KMLib_Connectors:1439890")
 		(at 99.822 184.912 0)
 		(unit 1)
@@
 	)
 	(symbol
-		(lib_id "kml-custom:1439890")
+		(lib_id "KMLib_Connectors:1439890")
 		(at 117.602 120.142 0)
 		(mirror y)
@@
 	)
 	(symbol
-		(lib_id "kml-custom:1439890")
+		(lib_id "KMLib_Connectors:1439890")
 		(at 99.822 98.552 0)
 		(unit 1)
