File: hardware/BREAD_Slice.kicad_sch (KiCad schematic)
At the start: 57 parts, among them IC1 ADS131M08IPBS, J1 Conn_01x10_Female, J10 Micro_SD_Card, J2 1439890, J3 1439890, J4 1439890, J5 1439890, J6 1439890, J7 1439890, J8 1439890, J9 1439890, U1 AP63205, U2 NUCLEO-L432KC, U3 MCP6022

Commit message: fix(hw): restore library prefixes on schematic Footprint properties
A symbol's Footprint property must be "Library:Item". These carried only the bare
item name, so KiCad reported a schematic/PCB parity error:

    KMLib_Connectors:1439890 doesn't match footprint given by symbol (1439890)

The prefix is taken from the PCB, which holds the full lib_id, matched by
reference designator -- not guessed. Symbols whose reference is absent from the
PCB, or whose PCB footprint has a different item name, were left alone.

No geometry changes; only the Footprint property text.

Schematic parity errors: 8 -> 0
Parts:
- J2, J3, J4, J5, J6, J7, J8, J9: footprint 1439890 -> KMLib_Connectors:1439890
Changed lines of the file:
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@@
 			)
 		)
-		(property "Footprint" "1439890"
+		(property "Footprint" "KMLib_Connectors:1439890"
 			(at 101.092 166.802 0)
 			(hide yes)
@@
 			)
 		)
-		(property "Footprint" "1439890"
+		(property "Footprint" "KMLib_Connectors:1439890"
 			(at 101.092 253.162 0)
 			(hide yes)
@@
 			)
 		)
-		(property "Footprint" "1439890"
+		(property "Footprint" "KMLib_Connectors:1439890"
 			(at 116.332 145.212 0)
 			(hide yes)
@@
 			)
 		)
-		(property "Footprint" "1439890"
+		(property "Footprint" "KMLib_Connectors:1439890"
 			(at 101.092 123.622 0)
 			(hide yes)
@@
 			)
 		)
-		(property "Footprint" "1439890"
+		(property "Footprint" "KMLib_Connectors:1439890"
 			(at 116.332 231.572 0)
 			(hide yes)
@@
 			)
 		)
-		(property "Footprint" "1439890"
+		(property "Footprint" "KMLib_Connectors:1439890"
 			(at 116.332 274.752 0)
 			(hide yes)
@@
 			)
 		)
-		(property "Footprint" "1439890"
+		(property "Footprint" "KMLib_Connectors:1439890"
 			(at 101.092 209.982 0)
 			(hide yes)
@@
 			)
 		)
-		(property "Footprint" "1439890"
+		(property "Footprint" "KMLib_Connectors:1439890"
 			(at 116.332 188.392 0)
 			(hide yes)
