File: hardware/fb_load_cell.kicad_sch (KiCad schematic)
At the start: 1 part

Commit message: final iteration of board with proper connectors and clean layout
Connections:
- net SHIELD: now also RSG1.5 (SHIELD); no longer RSG1.2 (SHIELD)
Changed lines of the file:
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@@
 		(pin "1"
 		)
-		(pin "2"
+		(pin "5"
 		)
 		(instances
