File: hardware/fb_load_cell.kicad_sch (KiCad schematic)
At the start: 1 part

Commit message: chore(hw): migrate KiCad files to the KiCad 10 format
Via `kicad-cli sch upgrade` / `pcb upgrade` (bread-infra
scripts/upgrade_kicad10.sh). Verified lossless: identical netlist, footprint
positions and routing.

Note `sch upgrade` does not cascade into hierarchical sub-sheets, so every
.kicad_sch is upgraded individually -- upgrading only the root sheet leaves
sub-sheets on the old format, which looks migrated and is not.
Parts:
- renumbered RSG1 to RSG3
Changed lines of the file:
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@@
 (kicad_sch
-	(version 20250114)
+	(version 20260306)
 	(generator "eeschema")
-	(generator_version "9.0")
+	(generator_version "10.0")
 	(paper "A4")
 	(wire
@@
 		(at 121.92 80.01 0)
 		(unit 1)
+		(body_style 1)
 		(exclude_from_sim no)
 		(in_bom no)
 		(on_board no)
+		(in_pos_files yes)
 		(dnp yes)
-		(property "Reference" "RSG1"
+		(property "Reference" "RSG3"
 			(at 118.11 82.804 0)
+			(show_name no)
+			(do_not_autoplace no)
 			(effects
 				(font
@@
 		(property "Value" "350"
 			(at 118.11 85.344 0)
+			(show_name no)
+			(do_not_autoplace no)
 			(effects
 				(font
@@
 		(property "Footprint" ""
 			(at 121.92 81.788 0)
+			(hide yes)
+			(show_name no)
+			(do_not_autoplace no)
 			(effects
 				(font
 					(size 1.27 1.27)
 				)
-				(hide yes)
 			)
 		)
-		(property "Datasheet" "~"
+		(property "Datasheet" ""
 			(at 121.92 80.01 0)
+			(hide yes)
+			(show_name no)
+			(do_not_autoplace no)
 			(effects
 				(font
 					(size 1.27 1.27)
 				)
-				(hide yes)
 			)
 		)
 		(property "Description" "Strain Gauge, Full Bridge"
 			(at 121.92 80.01 0)
+			(hide yes)
+			(show_name no)
+			(do_not_autoplace no)
 			(effects
 				(font
 					(size 1.27 1.27)
 				)
-				(hide yes)
 			)
 		)

Commit message: fix(hw): re-point stale library nicknames
These parts exist in KiCad-Master-Lib; the boards referenced libraries that no
longer exist (kml-custom, KML-Custom, and SparkFun libraries that never
contained the part) or names the library has since changed.

KiCad embeds footprint geometry in the .kicad_pcb, so the boards rendered and
fabricated correctly and the rot stayed invisible -- it only surfaces on
update-from-library, or when a generator tries to resolve a nickname.

Nickname/name only. No geometry is changed:

  SparkFun-DiscreteSemi:AP63205 -> KMLib_IC_Power:AP63205WU-7_Buck_Regulator
  SparkFun-LED:WS2812-5050-4PIN -> KMLib_IC_SMD:WS2812-5050-4PIN
  kml-custom:1439890 -> KMLib_Connectors:1439890
  kml-custom:AD8426BCPZ-WP -> KMLib_IC_Analog:AD8426BCPZ-WP_Instrumentation_Amplifier
  kml-custom:ADS131M08IPBS -> KMLib_IC_Analog:ADS131M08IPBS_24-bit_ADC
  kml-custom:CP_16_19_ADI -> KMLib_IC_SMD:CP_16_19_ADI
  kml-custom:DGN8_1P89X1P57 -> KMLib_IC_SMD:DGN8_1P89X1P57
  kml-custom:Full_Bridge_Strain_Gauge -> KMLib_Sensors:Full_Bridge_Strain_Gauge
  kml-custom:MODULE_NUCLEO-L432KC -> KMLib_Boards_Modules:MODULE_NUCLEO-L432KC
  kml-custom:NUCLEO-L432KC -> KMLib_IC_MCU_MPU:NUCLEO-L432KC
  kml-custom:QFP50P700X700X120-32N -> KMLib_IC_SMD:QFP50P700X700X120-32N
  kml-custom:TPS7A4901DGNR -> KMLib_IC_Power:TPS7A4901DGNR_LDO_Regulator
  kml-custom:Thermal Pad -> KMLib_Mounting:Thermal_Pad

Only references that failed to resolve were touched. Generic parts (<=4 pins)
and KiCad *-rescue libraries are deliberately excluded: fingerprint matching
cannot distinguish a 2-pin resistor from a 2-pin capacitor, so those are being
done by hand.
Parts:
- RSG3: symbol kml-custom:Full_Bridge_Strain_Gauge -> KMLib_Sensors:Full_Bridge_Strain_Gauge
Changed lines of the file:
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@@
 	)
 	(symbol
-		(lib_id "kml-custom:Full_Bridge_Strain_Gauge")
+		(lib_id "KMLib_Sensors:Full_Bridge_Strain_Gauge")
 		(at 121.92 80.01 0)
 		(unit 1)
